File: kicad_pcb/ergogen_pteron36_super/ergogen_pteron36_super.kicad_pcb (KiCad board)
At the start: 2 copper layers, 38 parts

Commit message: finalised config
Parts:
- added J1, J2: Jumper, lib:Jumper, F.Cu at (199.7, 106.7)
- added R1: R_0805, Resistor_SMD:R_0805_2012Metric_Pad1.20x1.40mm_HandSolder, F.Cu at (193.2, 164.2)
- added R2: R_0805, Resistor_SMD:R_0805_2012Metric_Pad1.20x1.40mm_HandSolder, F.Cu at (176.2, 164.2)
- moved MCU1 154.2 mm to (184.7, 120.7)
- moved FC1 150.1 mm to (184.7, 164.2)
- moved key12 141.4 mm to (131.6, 98.3)
- moved key11 141.4 mm to (125.1, 116.2)
- moved key21 141.4 mm to (299.8, 91.5)
- moved key24 141.4 mm to (273.1, 84.4)
- moved key29 141.4 mm to (244.2, 116.2)
- moved key3 141.4 mm to (69.6, 91.5)
- moved key6 141.4 mm to (96.3, 84.4)
- moved key30 141.4 mm to (237.7, 98.3)
- moved key15 141.4 mm to (148.8, 106.7)
- moved key16 141.4 mm to (130.2, 163.8)
- moved key18 141.4 mm to (158.1, 196.6)
- moved key4 141.4 mm to (83.3, 120.1)
- moved key5 141.4 mm to (89.8, 102.2)
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Other:
- board outline added: 277.1 x 141.5 mm
